File: esp32_picod4_downpads/esp32_picod4_downpads.sch (KiCad schematic (older format))
At the start: 84 parts, among them J1 PT0, J10 IO25, J11 IO26, J12 IO2, J13 MTDI, J14 EN, J15 IO0, J16 GND, J17 ‎2450AT42E0100E‎, J18 PGM_DBG, J19 Swadge_Parts_USB_B_Micro, J2 PT1, J3 PT2, J4 PT3, J5 PT4, J6 PT5, J7 PT6, J8 IO22, J9 IO23, K1 GND, K10 T6, K11 T7, K12 T8, K13 T9, K14 GND, K15 PT1, K16 PT2, K17 PT3, K18 PT4, K19 GND, K2 PT0, K20 3v3, K21 PT5, K22 G22, K23 G23, K24 G25, K25 G26, K26 PT6, K27 GND, K3 3v3, K4 ADC6, K5 ADC7, K6 GND, K7 T0, K8 T3, K9 T4, M1 GND, M2 GND, M3 GND, M4 GND, M5 GND, M6 GND, Q1 SS8050, Q2 SS8050, Q3 PMOS_GSD, Q4 PMOS_GSD, U1 ESP32-PICO-D4, U2 MCP1700-3302E_SOT23, U3 CP2104

Commit message: Forgot to upload design
Parts:
- removed J8: IO22, TestPoint:TestPoint_Pad_D1.5mm, symbol Connector_Generic:Conn_01x01
- removed M6: GND, MountingHole:MountingHole_3.2mm_M3_Pad_Via, symbol Connector_Generic:Conn_01x01
- removed R5, R6: 0, Resistor_SMD:R_0603_1608Metric, symbol Device:R_Small_US
- added K28: GND, TestPoint:TestPoint_Pad_D1.5mm, symbol Connector_Generic:Conn_01x01
- added L2: NC, Inductor_SMD:L_0603_1608Metric, symbol Device:L_Small
- K22: value G22 -> ANT
- U2: value MCP1700-3302E_SOT23 -> 3.3VREG
Connections:
- net GND: now also K28.1 (Pin_1)
- net GPIO22: no longer K22.1 (Pin_1)
- net at C3.2, L1.1, U1.2 (LNA_IN): now also L2.2
- net at U3.3 (D+): now also J19.3 (D+)
- net at U3.4 (D-): now also J19.2 (D-)
- new net: K22.1 (Pin_1), L2.1
Changed lines of the file:
@@
 Wire Wire Line
 	8700 4650 8850 4650
-$Comp
-L Device:R_Small_US R5
-U 1 1 5F259AAB
-P 8500 5150
-F 0 "R5" V 8400 5250 50  0000 C CNN
-F 1 "0" V 8400 5100 50  0000 C CNN
-F 2 "Resistor_SMD:R_0603_1608Metric" H 8500 5150 50  0001 C CNN
-F 3 "~" H 8500 5150 50  0001 C CNN
-	1    8500 5150
-	0    1    1    0
-$EndComp
-$Comp
-L Device:R_Small_US R6
-U 1 1 5F259F16
-P 8500 5250
-F 0 "R6" V 8400 5350 50  0000 C CNN
-F 1 "0" V 8400 5200 50  0000 C CNN
-F 2 "Resistor_SMD:R_0603_1608Metric" H 8500 5250 50  0001 C CNN
-F 3 "~" H 8500 5250 50  0001 C CNN
-	1    8500 5250
-	0    -1   -1   0
-$EndComp
-Wire Wire Line
-	8600 5250 8850 5250
-Wire Wire Line
-	8850 5150 8600 5150
-Wire Wire Line
-	8400 5150 8250 5150
-Wire Wire Line
-	8150 5250 8400 5250
 Text GLabel 4650 2850 2    50   Input ~ 0
 MTDI
@@
 ADC7
 $Comp
-L Connector_Generic:Conn_01x01 K22
-U 1 1 5F277C53
-P 1500 5300
-F 0 "K22" H 1800 5300 50  0000 C CNN
-F 1 "G22" H 1650 5300 50  0000 C CNN
-F 2 "TestPoint:TestPoint_Pad_D1.5mm" H 1500 5300 50  0001 C CNN
-F 3 "~" H 1500 5300 50  0001 C CNN
-	1    1500 5300
-	1    0    0    -1
-$EndComp
-$Comp
 L Connector_Generic:Conn_01x01 K23
 U 1 1 5F278043
@@
 Text GLabel 4650 3550 2    50   Input ~ 0
 GPIO22
-Text GLabel 2400 5200 2    50   Input ~ 0
-GPIO22
-$Comp
-L Connector_Generic:Conn_01x01 J8
-U 1 1 5F28F7B0
-P 2200 5200
-F 0 "J8" H 2118 4975 50  0000 C CNN
-F 1 "IO22" H 2118 5066 50  0000 C CNN
-F 2 "TestPoint:TestPoint_Pad_D1.5mm" H 2200 5200 50  0001 C CNN
-F 3 "~" H 2200 5200 50  0001 C CNN
-	1    2200 5200
-	-1   0    0    1
-$EndComp
 $Comp
 L Connector_Generic:Conn_01x01 K24
@@
 Text GLabel 1300 5400 0    50   Input ~ 0
 VSPIDGPIO23
-Text GLabel 1300 5300 0    50   Input ~ 0
-GPIO22
 $Comp
 L Connector_Generic:Conn_01x01 K27
@@
 P 5950 5950
 F 0 "U2" H 5950 6192 50  0000 C CNN
-F 1 "MCP1700-3302E_SOT23" H 5950 6101 50  0000 C CNN
+F 1 "3.3VREG" H 5950 6101 50  0000 C CNN
 F 2 "Package_TO_SOT_SMD:SOT-23" H 5950 6175 50  0001 C CNN
 F 3 "http://ww1.microchip.com/downloads/en/DeviceDoc/20001826D.pdf" H 5950 5950 50  0001 C CNN
@@
 F 3 "" H 1500 1100 50  0001 C CNN
 	1    1500 1100
-	0    -1   -1   0
-$EndComp
-$Comp
-L Connector_Generic:Conn_01x01 M6
-U 1 1 5F2D92B3
-P 1300 1500
-F 0 "M6" H 1218 1275 50  0000 C CNN
-F 1 "GND" H 1218 1366 50  0000 C CNN
-F 2 "MountingHole:MountingHole_3.2mm_M3_Pad_Via" H 1300 1500 50  0001 C CNN
-F 3 "~" H 1300 1500 50  0001 C CNN
-	1    1300 1500
-	-1   0    0    1
-$EndComp
-$Comp
-L power:GND #PWR013
-U 1 1 5F2D92B9
-P 1500 1500
-F 0 "#PWR013" H 1500 1250 50  0001 C CNN
-F 1 "GND" H 1505 1327 50  0000 C CNN
-F 2 "" H 1500 1500 50  0001 C CNN
-F 3 "" H 1500 1500 50  0001 C CNN
-	1    1500 1500
 	0    -1   -1   0
 $EndComp
@@
 Text Notes 850  6250 0    50   ~ 0
 1.5mm pads, staggered
+Wire Wire Line
+	8150 5250 8850 5250
+Wire Wire Line
+	8250 5150 8850 5150
+$Comp
+L Device:L_Small L2
+U 1 1 5F2BDE4A
+P 5200 1950
+F 0 "L2" V 5385 1950 50  0000 C CNN
+F 1 "NC" V 5294 1950 50  0000 C CNN
+F 2 "Inductor_SMD:L_0603_1608Metric" H 5200 1950 50  0001 C CNN
+F 3 "~" H 5200 1950 50  0001 C CNN
+	1    5200 1950
+	0    1    1    0
+$EndComp
+Wire Wire Line
+	5100 1950 5100 1850
+Connection ~ 5100 1850
+$Comp
+L Connector_Generic:Conn_01x01 K22
+U 1 1 5F2C11C3
+P 5500 1950
+F 0 "K22" H 5800 1950 50  0000 C CNN
+F 1 "ANT" H 5650 1950 50  0000 C CNN
+F 2 "TestPoint:TestPoint_Pad_D1.5mm" H 5500 1950 50  0001 C CNN
+F 3 "~" H 5500 1950 50  0001 C CNN
+	1    5500 1950
+	1    0    0    -1
+$EndComp
+$Comp
+L Connector_Generic:Conn_01x01 K28
+U 1 1 5F2DC71F
+P 1500 6600
+F 0 "K28" H 1800 6600 50  0000 C CNN
+F 1 "GND" H 1650 6600 50  0000 C CNN
+F 2 "TestPoint:TestPoint_Pad_D1.5mm" H 1500 6600 50  0001 C CNN
+F 3 "~" H 1500 6600 50  0001 C CNN
+	1    1500 6600
+	1    0    0    -1
+$EndComp
+$Comp
+L power:GND #PWR0108
+U 1 1 5F2DC725
+P 1300 6600
+F 0 "#PWR0108" H 1300 6350 50  0001 C CNN
+F 1 "GND" V 1300 6400 50  0000 C CNN
+F 2 "" H 1300 6600 50  0001 C CNN
+F 3 "" H 1300 6600 50  0001 C CNN
+	1    1300 6600
+	0    1    1    0
+$EndComp
 $EndSCHEMATC
