File: atmega168_tb2/atmega168_tb2.kicad_pcb (KiCad board)
At the start: 2 copper layers, 80 x 30 mm, 23 parts, among them J1 AVR-ISP-6, J2 WAVESHARE, J3 DBG_CARD, J4 Micro_SD_Card_Det, J5 BATT, J6 RX, J7 PE0, J8 PE1, J9 PE1, Q1 P_FET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

Commit message: bump.
Parts:
- J9: value PE1 -> GND
Other:
- board text added: "rev B"
- board text removed: "rev A"
Changed lines of the file:
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@@
-(kicad_pcb (version 20171130) (host pcbnew 5.1.6-c6e7f7d~86~ubuntu18.04.1)
+(kicad_pcb (version 20171130) (host pcbnew 5.1.6-c6e7f7d~87~ubuntu18.04.1)
   (general
     (thickness 1.6)
@@
       (effects (font (size 1 1) (thickness 0.15)))
     )
-    (fp_text user %R (at 0 -2.15) (layer F.Fab)
-      (effects (font (size 1 1) (thickness 0.15)))
-    )
     (fp_line (start -1.45 -1.45) (end 1.45 -1.45) (layer F.SilkS) (width 0.12))
     (fp_line (start 1.45 -1.45) (end 1.45 1.45) (layer F.SilkS) (width 0.12))
@@
     (fp_line (start 1.75 1.75) (end 1.75 -1.75) (layer F.CrtYd) (width 0.05))
     (fp_line (start 1.75 1.75) (end -1.75 1.75) (layer F.CrtYd) (width 0.05))
+    (fp_text user %R (at 0 -2.15) (layer F.Fab)
+      (effects (font (size 1 1) (thickness 0.15)))
+    )
     (pad 1 smd rect (at 0 0) (size 2.5 2.5) (layers F.Cu F.Mask)
       (net 31 RX))
@@
     )
     (fp_text value PE1 (at 0 2.25) (layer F.SilkS)
-      (effects (font (size 1 1) (thickness 0.15)))
-    )
-    (fp_text user %R (at 0 -2.15) (layer F.Fab)
       (effects (font (size 1 1) (thickness 0.15)))
     )
@@
     (fp_line (start 1.75 1.75) (end 1.75 -1.75) (layer F.CrtYd) (width 0.05))
     (fp_line (start 1.75 1.75) (end -1.75 1.75) (layer F.CrtYd) (width 0.05))
+    (fp_text user %R (at 0 -2.15) (layer F.Fab)
+      (effects (font (size 1 1) (thickness 0.15)))
+    )
     (pad 1 smd rect (at 0 0) (size 2.5 2.5) (layers F.Cu F.Mask)
       (net 33 PE1))
@@
       (effects (font (size 1 1) (thickness 0.15)))
     )
-    (fp_text value PE1 (at 0.06 2.67) (layer F.SilkS)
+    (fp_text value GND (at 0.06 2.67) (layer F.SilkS)
       (effects (font (size 1 1) (thickness 0.15)))
     )
@@
       (net 2 GND))
   )
-  (gr_text "rev A" (at 115.835 49.905) (layer F.SilkS)
+  (gr_text "rev B" (at 115.835 49.905) (layer F.SilkS)
     (effects (font (size 1 1) (thickness 0.15)))
   )
