File: atmega168_tb2/atmega168_tb2.sch (KiCad schematic (older format))
At the start: 23 parts, among them J1 AVR-ISP-6, J2 WAVESHARE, J3 DBG_CARD, J4 Micro_SD_Card_Det, J5 BATT, J6 RX, J7 PE0, J8 PE1, J9 PE1, Q1 P_FET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

Commit message: bump.
Parts:
- C1, C2, C3, C4, C5, C6, C7: symbol Device:C_Small -> atmega168_tb2-rescue:C_Small-Device
- J1: symbol Connector:AVR-ISP-6 -> atmega168_tb2-rescue:AVR-ISP-6-Connector
- J2: symbol Connector_Generic:Conn_01x08 -> atmega168_tb2-rescue:Conn_01x08-Connector_Generic
- J3: symbol Connector_Generic:Conn_01x10 -> atmega168_tb2-rescue:Conn_01x10-Connector_Generic
- J4: symbol Connector:Micro_SD_Card_Det -> atmega168_tb2-rescue:Micro_SD_Card_Det-Connector
- J5: symbol Connector_Generic:Conn_01x02 -> atmega168_tb2-rescue:Conn_01x02-Connector_Generic
- J6, J7, J8: symbol Connector:Conn_01x01_Female -> atmega168_tb2-rescue:Conn_01x01_Female-Connector
- J9: value PE1 -> GND; symbol Connector:Conn_01x01_Female -> atmega168_tb2-rescue:Conn_01x01_Female-Connector
- Q1, Q2: symbol Device:Q_PMOS_GSD -> atmega168_tb2-rescue:Q_PMOS_GSD-Device
- R1, R2: symbol Device:R_Small -> atmega168_tb2-rescue:R_Small-Device
- U1: symbol Regulator_Linear:LP2985-3.0 -> atmega168_tb2-rescue:LP2985-3.0-Regulator_Linear
- U2: symbol MCU_Microchip_ATmega:ATmega168PB-AU -> atmega168_tb2-rescue:ATmega168PB-AU-MCU_Microchip_ATmega
- Y1: symbol Device:Crystal -> atmega168_tb2-rescue:Crystal-Device
Changed lines of the file:
@@
 $EndDescr
 $Comp
-L MCU_Microchip_ATmega:ATmega168PB-AU U2
+L atmega168_tb2-rescue:ATmega168PB-AU-MCU_Microchip_ATmega U2
 U 1 1 5F1D38A0
 P 3550 2950
@@
 $EndComp
 $Comp
-L power:GND #PWR0101
+L atmega168_tb2-rescue:GND-power #PWR0101
 U 1 1 5F1D3F0C
 P 3550 4450
@@
 $EndComp
 $Comp
-L power:+BATT #PWR0102
+L atmega168_tb2-rescue:+BATT-power #PWR0102
 U 1 1 5F1D483B
 P 3650 1450
@@
 $EndComp
 $Comp
-L power:+BATT #PWR0103
+L atmega168_tb2-rescue:+BATT-power #PWR0103
 U 1 1 5F1D4C41
 P 3550 1450
@@
 $EndComp
 $Comp
-L power:+BATT #PWR0104
+L atmega168_tb2-rescue:+BATT-power #PWR0104
 U 1 1 5F1D4F57
 P 1600 1950
@@
 $EndComp
 $Comp
-L Connector:Micro_SD_Card_Det J4
+L atmega168_tb2-rescue:Micro_SD_Card_Det-Connector J4
 U 1 1 5F1D5A97
 P 8350 2400
@@
 $EndComp
 $Comp
-L power:GND #PWR0105
+L atmega168_tb2-rescue:GND-power #PWR0105
 U 1 1 5F1D68C8
 P 9150 2900
@@
 $EndComp
 $Comp
-L Device:Crystal Y1
+L atmega168_tb2-rescue:Crystal-Device Y1
 U 1 1 5F1DD35C
 P 5150 2400
@@
 	4900 2550 5150 2550
 $Comp
-L Device:C_Small C2
+L atmega168_tb2-rescue:C_Small-Device C2
 U 1 1 5F1DDFF0
 P 4900 2650
@@
 Connection ~ 5150 2250
 $Comp
-L Device:C_Small C5
+L atmega168_tb2-rescue:C_Small-Device C5
 U 1 1 5F1DEE70
 P 5550 2650
@@
 $EndComp
 $Comp
-L power:GND #PWR0106
+L atmega168_tb2-rescue:GND-power #PWR0106
 U 1 1 5F1DF1D9
 P 5550 2750
@@
 $EndComp
 $Comp
-L power:GND #PWR0107
+L atmega168_tb2-rescue:GND-power #PWR0107
 U 1 1 5F1DF5B0
 P 4900 2750
@@
 $EndComp
 $Comp
-L power:GND #PWR0108
+L atmega168_tb2-rescue:GND-power #PWR0108
 U 1 1 5F1DF898
 P 4150 1950
@@
 $EndComp
 $Comp
-L power:+BATT #PWR0109
+L atmega168_tb2-rescue:+BATT-power #PWR0109
 U 1 1 5F1E0230
 P 6200 3650
@@
 CARD_VDD
 $Comp
-L Device:Q_PMOS_GSD Q2
+L atmega168_tb2-rescue:Q_PMOS_GSD-Device Q2
 U 1 1 5F1E285C
 P 6600 3750
@@
 CARDCLK
 $Comp
-L power:GND #PWR0110
+L atmega168_tb2-rescue:GND-power #PWR0110
 U 1 1 5F1E5CF5
 P 7450 2500
@@
 CARD_DET
 $Comp
-L Connector:AVR-ISP-6 J1
+L atmega168_tb2-rescue:AVR-ISP-6-Connector J1
 U 1 1 5F207105
 P 1100 3300
@@
 $EndComp
 $Comp
-L power:GND #PWR0111
+L atmega168_tb2-rescue:GND-power #PWR0111
 U 1 1 5F2076C1
 P 1000 3700
@@
 MISO
 $Comp
-L Regulator_Linear:LP2985-3.0 U1
+L atmega168_tb2-rescue:LP2985-3.0-Regulator_Linear U1
 U 1 1 5F209147
 P 1200 2050
@@
 $EndComp
 $Comp
-L power:GND #PWR0112
+L atmega168_tb2-rescue:GND-power #PWR0112
 U 1 1 5F209AC4
 P 1200 2350
@@
 RST
 $Comp
-L Device:C_Small C4
+L atmega168_tb2-rescue:C_Small-Device C4
 U 1 1 5F212E37
 P 5350 3800
@@
 $EndComp
 $Comp
-L power:GND #PWR0113
+L atmega168_tb2-rescue:GND-power #PWR0113
 U 1 1 5F2134AA
 P 5350 3900
@@
 $EndComp
 $Comp
-L Device:C_Small C3
+L atmega168_tb2-rescue:C_Small-Device C3
 U 1 1 5F2145C2
 P 5000 3800
@@
 $EndComp
 $Comp
-L power:+BATT #PWR0114
+L atmega168_tb2-rescue:+BATT-power #PWR0114
 U 1 1 5F2149DF
 P 5000 3700
@@
 $EndComp
 $Comp
-L Device:C_Small C6
+L atmega168_tb2-rescue:C_Small-Device C6
 U 1 1 5F214E68
 P 5750 3800
@@
 $EndComp
 $Comp
-L power:+BATT #PWR0115
+L atmega168_tb2-rescue:+BATT-power #PWR0115
 U 1 1 5F215340
 P 5750 3700
@@
 $EndComp
 $Comp
-L power:GND #PWR0116
+L atmega168_tb2-rescue:GND-power #PWR0116
 U 1 1 5F215811
 P 5000 3900
@@
 $EndComp
 $Comp
-L power:GND #PWR0117
+L atmega168_tb2-rescue:GND-power #PWR0117
 U 1 1 5F215C86
 P 5750 3900
@@
 $EndComp
 $Comp
-L Device:C_Small C7
+L atmega168_tb2-rescue:C_Small-Device C7
 U 1 1 5F21618B
 P 7550 3700
@@
 CARD_VDD
 $Comp
-L power:GND #PWR0118
+L atmega168_tb2-rescue:GND-power #PWR0118
 U 1 1 5F2169DC
 P 7550 3800
@@
 CARDPWR
 $Comp
-L Device:R_Small R1
+L atmega168_tb2-rescue:R_Small-Device R1
 U 1 1 5F2175BB
 P 7150 4250
@@
 $EndComp
 $Comp
-L power:+BATT #PWR0119
+L atmega168_tb2-rescue:+BATT-power #PWR0119
 U 1 1 5F21AD24
 P 7150 4150
@@
 $EndComp
 $Comp
-L Connector_Generic:Conn_01x10 J3
+L atmega168_tb2-rescue:Conn_01x10-Connector_Generic J3
 U 1 1 5F221146
 P 6550 2400
@@
 $EndComp
 $Comp
-L power:GND #PWR0120
+L atmega168_tb2-rescue:GND-power #PWR0120
 U 1 1 5F222CB0
 P 6350 2900
@@
 CARDCLK
 $Comp
-L power:+BATT #PWR0121
+L atmega168_tb2-rescue:+BATT-power #PWR0121
 U 1 1 5F22ABC2
 P 6350 2000
@@
 $EndComp
 $Comp
-L power:+5V #PWR0122
+L atmega168_tb2-rescue:+5V-power #PWR0122
 U 1 1 5F22B725
 P 850 2800
@@
 	850  2800 1000 2800
 $Comp
-L power:+5V #PWR0123
+L atmega168_tb2-rescue:+5V-power #PWR0123
 U 1 1 5F22BD41
 P 6350 2100
@@
 CARD_VDD
 $Comp
-L Connector_Generic:Conn_01x08 J2
+L atmega168_tb2-rescue:Conn_01x08-Connector_Generic J2
 U 1 1 5F2507D9
 P 5200 4950
@@
 PDI
 $Comp
-L power:GND #PWR0124
+L atmega168_tb2-rescue:GND-power #PWR0124
 U 1 1 5F260FC1
 P 5000 5250
@@
 $EndComp
 $Comp
-L Device:Q_PMOS_GSD Q1
+L atmega168_tb2-rescue:Q_PMOS_GSD-Device Q1
 U 1 1 5F261447
 P 4100 5450
@@
 PPWRCTRL
 $Comp
-L power:+BATT #PWR0125
+L atmega168_tb2-rescue:+BATT-power #PWR0125
 U 1 1 5F262E50
 P 3900 5350
@@
 PPWRCTRL
 $Comp
-L Device:C_Small C1
+L atmega168_tb2-rescue:C_Small-Device C1
 U 1 1 5F26D062
 P 1900 4400
@@
 $EndComp
 $Comp
-L power:GND #PWR0126
+L atmega168_tb2-rescue:GND-power #PWR0126
 U 1 1 5F26D557
 P 1900 4500
@@
 $EndComp
 $Comp
-L power:+BATT #PWR0127
+L atmega168_tb2-rescue:+BATT-power #PWR0127
 U 1 1 5F26DAD5
 P 1900 4300
@@
 $EndComp
 $Comp
-L Device:R_Small R2
+L atmega168_tb2-rescue:R_Small-Device R2
 U 1 1 5F27AEF3
 P 3050 5500
@@
 PPWRCTRL
 $Comp
-L power:+BATT #PWR0128
+L atmega168_tb2-rescue:+BATT-power #PWR0128
 U 1 1 5F27BFC3
 P 3050 5400
@@
 $EndComp
 $Comp
-L Connector_Generic:Conn_01x02 J5
+L atmega168_tb2-rescue:Conn_01x02-Connector_Generic J5
 U 1 1 5F287D5B
 P 6300 4650
@@
 $EndComp
 $Comp
-L power:GND #PWR0129
+L atmega168_tb2-rescue:GND-power #PWR0129
 U 1 1 5F288244
 P 6100 4750
@@
 $EndComp
 $Comp
-L power:+BATT #PWR0130
+L atmega168_tb2-rescue:+BATT-power #PWR0130
 U 1 1 5F288895
 P 6100 4650
@@
 PE1
 $Comp
-L Connector:Conn_01x01_Female J6
+L atmega168_tb2-rescue:Conn_01x01_Female-Connector J6
 U 1 1 5F205323
 P 5200 1200
@@
 $EndComp
 $Comp
-L Connector:Conn_01x01_Female J7
+L atmega168_tb2-rescue:Conn_01x01_Female-Connector J7
 U 1 1 5F206AE0
 P 5200 1400
@@
 $EndComp
 $Comp
-L Connector:Conn_01x01_Female J8
+L atmega168_tb2-rescue:Conn_01x01_Female-Connector J8
 U 1 1 5F2077A2
 P 5200 1600
@@
 RX
 $Comp
-L Connector:Conn_01x01_Female J9
+L atmega168_tb2-rescue:Conn_01x01_Female-Connector J9
 U 1 1 5F208BCE
 P 5200 1800
 F 0 "J9" H 5228 1826 50  0000 L CNN
-F 1 "PE1" H 5228 1735 50  0000 L CNN
+F 1 "GND" H 5228 1735 50  0000 L CNN
 F 2 "TestPoint:TestPoint_Pad_2.5x2.5mm" H 5200 1800 50  0001 C CNN
 F 3 "~" H 5200 1800 50  0001 C CNN
@@
 $EndComp
 $Comp
-L power:GND #PWR0131
+L atmega168_tb2-rescue:GND-power #PWR0131
 U 1 1 5F20BC57
 P 5000 1800
